Commit message: barista sdf

File: barista_description/src/description/barista.urdf (robot description, URDF)
Before this commit: robot barista, 31 links, 30 joints
Joints:
- removed joint joint_tire_left
- removed joint joint_tire_right
- added joint wheel_left_joint: type continuous, parent base_link, child wheel_left_link, origin xyz=0.00 0.115 0.0250 rpy=-1.5707963267948966 0 0, axis 0 0 1
- added joint wheel_right_joint: type continuous, parent base_link, child wheel_right_link, origin xyz=0.00 -0.115 0.0250 rpy=-1.5707963267948966 0 0, axis 0 0 1

Commit message: slotcar plugin working, gazebo spawns sdf file

File: barista_description/src/description/barista.urdf (robot description, URDF)
Before this commit: robot barista, 31 links, 30 joints
Links:
- link barista_bottom_link: geometry collision cylinder length=0.14 radius=0.1760015; visual mesh filename=package://barista_description/meshes/barista/BOTTOM_colour.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
- link barista_bowtie_link: geometry collision box size=0.115703 0.024221 0.0589962; visual mesh filename=package://barista_description/meshes/barista/bowtie_fixed_c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
- link barista_top_link: geometry collision cylinder length=0.085 radius=0.1760015; visual mesh filename=package://barista_description/meshes/barista/TOP_colour.dae
- link base_link: geometry collision cylinder length=0.10938 radius=0.178; visual mesh filename=package://barista_description/meshes/main_body.dae
- link laser_sensor_link: geometry collision box size=0.1 0.1 0.1; visual mesh filename=package://barista_description/meshes/sensors/hokuyo.dae
- link plate_bottom_link: geometry collision cylinder length=0.006 radius=0.170; visual mesh filename=package://barista_description/meshes/stacks/hexagons/plate_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
- link plate_middle_link: geometry collision cylinder length=0.006 radius=0.170; visual mesh filename=package://barista_description/meshes/stacks/hexagons/plate_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
- link plate_top_link: geometry collision cylinder length=0.006 radius=0.170; visual mesh filename=package://barista_description/meshes/stacks/hexagons/plate_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
- link pole_bottom_0_link: geometry collision cylinder length=0.0492 radius=0.006; visual mesh filename=package://barista_description/meshes/stacks/hexagons/pole_b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
- link pole_bottom_1_link: geometry collision cylinder length=0.0492 radius=0.006; visual mesh filename=package://barista_description/meshes/stacks/hexagons/pole_b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
- link pole_bottom_2_link: geometry collision cylinder length=0.0492 radius=0.006; visual mesh filename=package://barista_description/meshes/stacks/hexagons/pole_b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
- link pole_bottom_3_link: geometry collision cylinder length=0.0492 radius=0.006; visual mesh filename=package://barista_description/meshes/stacks/hexagons/pole_b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
- link pole_bottom_4_link: geometry collision cylinder length=0.0492 radius=0.006; visual mesh filename=package://barista_description/meshes/stacks/hexagons/pole_b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
- link pole_bottom_5_link: geometry collision cylinder length=0.0492 radius=0.006; visual mesh filename=package://barista_description/meshes/stacks/hexagons/pole_b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
- link pole_middle_0_link: geometry collision cylinder length=0.0608 radius=0.006; visual mesh filename=package://barista_description/meshes/stacks/hexagons/pole_m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
- link pole_middle_1_link: geometry collision cylinder length=0.0608 radius=0.006; visual mesh filename=package://barista_description/meshes/stacks/hexagons/pole_m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
- link pole_middle_2_link: geometry collision cylinder length=0.0608 radius=0.006; visual mesh filename=package://barista_description/meshes/stacks/hexagons/pole_m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
- link pole_middle_3_link: geometry collision cylinder length=0.0608 radius=0.006; visual mesh filename=package://barista_description/meshes/stacks/hexagons/pole_m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
- link pole_top_0_link: geometry collision cylinder length=0.2032 radius=0.006; visual mesh filename=package://barista_description/meshes/stacks/hexagons/pole_t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
- link pole_top_1_link: geometry collision cylinder length=0.2032 radius=0.006; visual mesh filename=package://barista_description/meshes/stacks/hexagons/pole_t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
- link pole_top_2_link: geometry collision cylinder length=0.2032 radius=0.006; visual mesh filename=package://barista_description/meshes/stacks/hexagons/pole_t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
- link pole_top_3_link: geometry collision cylinder length=0.2032 radius=0.006; visual mesh filename=package://barista_description/meshes/stacks/hexagons/pole_t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
- link wheel_left_link: geometry collision cylinder length=0.0206 radius=0.0352; visual mesh filename=package://barista_description/meshes/wheel.dae
- link wheel_right_link: geometry collision cylinder length=0.0206 radius=0.0350; visual mesh filename=package://barista_description/meshes/wheel.dae
Joints:
- removed joint wheel_left_joint
- removed joint wheel_right_joint
- added joint joint_tire_left: type continuous, parent base_link, child wheel_left_link, origin xyz=0.00 0.115 0.0250 rpy=-1.5707963267948966 0 0, axis 0 0 1
- added joint joint_tire_right: type continuous, parent base_link, child wheel_right_link, origin xyz=0.00 -0.115 0.0250 rpy=-1.5707963267948966 0 0, axis 0 0 1
