Commit message: latest changes

File: barista_description/robot/barista.xacro (robot description, xacro)
@@ -10,5 +10,5 @@
   <xacro:include filename="$(find barista_description)/robot/barista_mod.xacro" />
   <xacro:include filename="$(find barista_description)/robot/barista_hokuyo.xacro" />
-  <xacro:barista_kobuki/>
+  <xacro:barista_kobuki robot_name="$(arg robot_name)"/>
   <xacro:stack_hexagons parent="base_link"/>
   <xacro:barista_mod  bottom_parent="plate_middle_link" top_parent="plate_top_link"/>

File: barista_description/robot/barista_hokuyo.xacro (robot description, xacro)
@@ -59,11 +59,36 @@
 			<plugin name="scan" filename="libgazebo_ros_ray_sensor.so">
 				<ros>
+					<namespace>${robot_name}</namespace>
 					<remapping>~/out:=scan</remapping>
 				</ros>
 				<output_type>sensor_msgs/LaserScan</output_type>
-				<frame_name>laser_sensor_link</frame_name>
+				<frame_name>${robot_name}/laser_sensor_link</frame_name>
 			</plugin>
 		</sensor>
   	</gazebo>
+	<gazebo>
+		<plugin name='diff_drive' filename='libgazebo_ros_diff_drive.so'>
+			<ros>
+				<namespace>/</namespace>
+				<argument>cmd_vel:=${robot_name}/cmd_vel</argument>
+				<argument>odom:=${robot_name}/odom</argument>
+			</ros>
+			<!-- wheels -->
+			<left_joint>${robot_name}/joint_tire_left</left_joint>
+			<right_joint>${robot_name}/joint_tire_right</right_joint>
+			<!-- kinematics -->
+			<wheel_separation>0.4</wheel_separation>
+			<wheel_diameter>0.1</wheel_diameter>
+			<!-- limits -->
+			<max_wheel_torque>20</max_wheel_torque>
+			<max_wheel_acceleration>1.0</max_wheel_acceleration>
+			<!-- output -->
+			<publish_odom>true</publish_odom>
+			<publish_odom_tf>true</publish_odom_tf>
+			<publish_wheel_tf>false</publish_wheel_tf>
+			<odometry_frame>odom</odometry_frame>
+			<robot_base_frame>${robot_name}/base_footprint</robot_base_frame>
+		</plugin>
+	</gazebo>
   </xacro:macro>
 </robot>

File: barista_description/robot/barista_kobuki.xacro (robot description, xacro)
@@ -1,8 +1,9 @@
 <?xml version="1.0" ?>
 <robot name="barista_kobuki" xmlns:xacro="http://ros.org/wiki/xacro">
+  <xacro:arg name="robot_name" default="barista_X"/>
   <xacro:include filename="$(find barista_description)/robot/kobuki/common_properties.urdf.xacro"/>
   <xacro:include filename="$(find barista_description)/robot/barista_kobuki_gazebo.xacro"/>
   <!-- Kobuki -->
-  <xacro:macro name="barista_kobuki">
+  <xacro:macro name="barista_kobuki" params="robot_name">
     <link name="base_footprint"/>
     <joint name="base_joint" type="fixed">
@@ -34,11 +35,11 @@
       </inertial>
     </link>
-    <joint name="joint_tire_left" type="continuous">
+    <joint name="${robot_name}/joint_tire_left" type="continuous">
     <parent link="base_link"/>
-    <child link="wheel_left_link"/>
+    <child link="${robot_name}/wheel_left_link"/>
     <origin rpy="-1.5707963267948966 0 0" xyz="0.00 0.115 0.0250"/>
     <axis xyz="0 0 1"/>
   </joint>
-  <link name="wheel_left_link">
+  <link name="${robot_name}/wheel_left_link">
     <visual>
       <geometry>
@@ -59,11 +60,11 @@
     </inertial>
   </link>
-  <joint name="joint_tire_right" type="continuous">
+  <joint name="${robot_name}/joint_tire_right" type="continuous">
     <parent link="base_link"/>
-    <child link="wheel_right_link"/>
+    <child link="${robot_name}/wheel_right_link"/>
     <origin rpy="-1.5707963267948966 0 0" xyz="0.00 -0.115 0.0250"/>
     <axis xyz="0 0 1"/>
   </joint>
-  <link name="wheel_right_link">
+  <link name="${robot_name}/wheel_right_link">
     <visual>
       <geometry>
@@ -183,5 +184,5 @@
     </link>
     <!-- Kobuki Gazebo simulation details -->
-    <xacro:kobuki_sim/>
+    <xacro:kobuki_sim robot_name="$(arg robot_name)"/>
   </xacro:macro>
 </robot>

File: barista_description/robot/barista_kobuki_gazebo.xacro (robot description, xacro)
@@ -1,5 +1,6 @@
 <?xml version="1.0"?>
 <robot name="kobuki_sim" xmlns:xacro="http://ros.org/wiki/xacro">
-  <xacro:macro name="kobuki_sim">
+  <xacro:arg name="robot_name" default="barista_X"/>
+  <xacro:macro name="kobuki_sim" params="robot_name">
 	  <gazebo reference="wheel_left_link">
 	    <mu1>1.0</mu1>
@@ -136,26 +137,4 @@
       </sensor>
 	  </gazebo>
-	<gazebo>
-		<plugin name='diff_drive' filename='libgazebo_ros_diff_drive.so'>
-			<ros>
-				<namespace>/</namespace>
-			</ros>
-			<!-- wheels -->
-			<left_joint>joint_tire_left</left_joint>
-			<right_joint>joint_tire_right</right_joint>
-			<!-- kinematics -->
-			<wheel_separation>0.4</wheel_separation>
-			<wheel_diameter>0.1</wheel_diameter>
-			<!-- limits -->
-			<max_wheel_torque>20</max_wheel_torque>
-			<max_wheel_acceleration>1.0</max_wheel_acceleration>
-			<!-- output -->
-			<publish_odom>true</publish_odom>
-			<publish_odom_tf>true</publish_odom_tf>
-			<publish_wheel_tf>true</publish_wheel_tf>
-			<odometry_frame>odom</odometry_frame>
-			<robot_base_frame>base_footprint</robot_base_frame>
-		</plugin>
-	</gazebo>
   </xacro:macro>
 </robot>
