Commit message: Added mods for deliver demo

File: barista_description/robot/barista_mod.xacro (robot description, xacro)
@@ -22,7 +22,9 @@
       </visual>
       <collision>
-        <origin xyz="-0.0425 0 0" rpy="0 0 0"/>
+        <origin xyz="0 0 0" rpy="0 0 0"/>
+        <!-- <origin xyz="-0.0425 0 0" rpy="0 0 0"/> -->
         <geometry>
-          <cylinder length="0.085" radius="0.1760015"/>
+          <mesh filename="package://barista_description/meshes/barista/TOP_collision_lip.stl"/>
+          <!-- <cylinder length="0.085" radius="0.1760015"/> -->
         </geometry>
       </collision>
