Commit message: Added new mule version

File: barista_description/robot/barista_hexagons.xacro (robot description, xacro)
@@ -127,4 +127,40 @@
   -->
   <xacro:macro name="stack_hexagons" params="parent">
+    <xacro:stack_hexagons_base parent="${parent}"/>
+    <xacro:stack_hexagons_top parent="${parent}"/>
+  </xacro:macro>
+  <xacro:macro name="stack_hexagons_top" params="parent">
+    <xacro:stack_top_pole parent="${parent}" number="0" x_loc= "0.0381" y_loc= "0.1505" z_loc="0.2920"/>
+    <xacro:stack_top_pole parent="${parent}" number="1" x_loc= "0.0381" y_loc="-0.1505" z_loc="0.2920"/>
+    <xacro:stack_top_pole parent="${parent}" number="2" x_loc="-0.0381" y_loc= "0.1505" z_loc="0.2920"/>
+    <xacro:stack_top_pole parent="${parent}" number="3" x_loc="-0.0381" y_loc="-0.1505" z_loc="0.2920"/>
+    <joint name="plate_top_joint" type="fixed">
+      <origin xyz="-0.01364 0.0  0.3966" rpy="0 0 0"/>
+      <parent link="${parent}"/>
+      <child link="plate_top_link"/>
+    </joint>
+    <link name="plate_top_link">
+      <visual>
+        <origin xyz="0 0 0" rpy="0 0 0"/>
+        <geometry>
+          <mesh filename="package://barista_description/meshes/stacks/hexagons/plate_top.dae"/>
+        </geometry>
+      </visual>
+      <collision>
+        <origin xyz="0.01364 0 0" rpy="0 0 0"/>
+        <geometry>
+          <cylinder length="0.006" radius="0.170"/>
+        </geometry>
+      </collision>
+      <inertial>
+        <mass value="0.520"/>
+        <origin xyz="0 0 0"/>
+        <inertia ixx="0.003328" ixy="0.0" ixz="0.0"
+                 iyy="0.003328" iyz="0.0"
+                 izz="0.006656" />
+      </inertial>
+    </link>
+  </xacro:macro>
+  <xacro:macro name="stack_hexagons_base" params="parent">
     <xacro:stack_bottom_pole parent="${parent}" number="0" x_loc= "0.120" y_loc= "0.082" z_loc="0.1028"/>
     <xacro:stack_bottom_pole parent="${parent}" number="1" x_loc= "0.055" y_loc= "0.120" z_loc="0.1028"/>
@@ -189,38 +225,15 @@
       </inertial>
     </link>
-    <xacro:stack_top_pole parent="${parent}" number="0" x_loc= "0.0381" y_loc= "0.1505" z_loc="0.2920"/>
-    <xacro:stack_top_pole parent="${parent}" number="1" x_loc= "0.0381" y_loc="-0.1505" z_loc="0.2920"/>
-    <xacro:stack_top_pole parent="${parent}" number="2" x_loc="-0.0381" y_loc= "0.1505" z_loc="0.2920"/>
-    <xacro:stack_top_pole parent="${parent}" number="3" x_loc="-0.0381" y_loc="-0.1505" z_loc="0.2920"/>
-    <!--
-    <stack_3d_sensor_pole parent="${parent}" number="0" x_loc="-0.1024" y_loc= "0.098" z_loc="0.2372"/>
-    <stack_3d_sensor_pole parent="${parent}" number="1" x_loc="-0.1024" y_loc="-0.098" z_loc="0.2372"/>
-    -->
-    <joint name="plate_top_joint" type="fixed">
-      <origin xyz="-0.01364 0.0  0.3966" rpy="0 0 0"/>
-      <parent link="${parent}"/>
-      <child link="plate_top_link"/>
-    </joint>
-    <link name="plate_top_link">
-      <visual>
-        <origin xyz="0 0 0" rpy="0 0 0"/>
-        <geometry>
-          <mesh filename="package://barista_description/meshes/stacks/hexagons/plate_top.dae"/>
-        </geometry>
-      </visual>
-      <collision>
-        <origin xyz="0.01364 0 0" rpy="0 0 0"/>
-        <geometry>
-          <cylinder length="0.006" radius="0.170"/>
-        </geometry>
-      </collision>
-      <inertial>
-        <mass value="0.520"/>
-        <origin xyz="0 0 0"/>
-        <inertia ixx="0.003328" ixy="0.0" ixz="0.0"
-                 iyy="0.003328" iyz="0.0"
-                 izz="0.006656" />
-      </inertial>
-    </link>
+  </xacro:macro>
+  <!-- MULE Barista related mods -->
+    <xacro:macro name="stack_hexagons_mule" params="parent">
+    <xacro:stack_hexagons_base parent="${parent}"/>
+    <xacro:stack_hexagons_top_mule parent="${parent}"/>
+  </xacro:macro>
+  <xacro:macro name="stack_hexagons_top_mule" params="parent">
+    <xacro:stack_middle_pole parent="${parent}" number="4" x_loc= "0.0381" y_loc= "0.1505" z_loc="0.2570"/>
+    <xacro:stack_middle_pole parent="${parent}" number="5" x_loc= "0.0381" y_loc="-0.1505" z_loc="0.2570"/>
+    <xacro:stack_middle_pole parent="${parent}" number="6" x_loc="-0.0381" y_loc= "0.1505" z_loc="0.2570"/>
+    <xacro:stack_middle_pole parent="${parent}" number="7" x_loc="-0.0381" y_loc="-0.1505" z_loc="0.2570"/>
   </xacro:macro>
 </robot>

File: barista_description/robot/barista_mod.xacro (robot description, xacro)
@@ -5,10 +5,18 @@
 <robot name="stack_hexagons" xmlns:xacro="http://ros.org/wiki/xacro">
   <xacro:include filename="$(find barista_description)/robot/turtlebot/common_properties.urdf.xacro"/>
-  <xacro:macro name="barista_mod" params="bottom_parent top_parent">
+  <xacro:macro name="barista_mod" params="bottom_parent top_parent ">
     <link name="barista_top_link">
       <visual>
         <origin xyz="0 0 0" rpy="0 0 0"/>
         <geometry>
-          <mesh filename="package://barista_description/meshes/barista/TOP_colour.dae"/>
+          <xacro:if value="${robot_name_prop == 'barista_1'}">
+            <mesh filename="package://barista_description/meshes/barista/TOP_colour_1.dae"/>
+          </xacro:if>
+          <xacro:if value="${robot_name_prop == 'barista_2'}">
+            <mesh filename="package://barista_description/meshes/barista/TOP_colour_2.dae"/>
+          </xacro:if>
+          <xacro:if value="${robot_name_prop != 'barista_1' and robot_name_prop != 'barista_2'}">
+            <mesh filename="package://barista_description/meshes/barista/TOP_colour.dae"/>
+          </xacro:if>
         </geometry>
       </visual>
@@ -32,29 +40,66 @@
       <child link="barista_top_link"/>
     </joint>
-    <link name="barista_bowtie_link">
+    <link name="barista_bottom_link">
       <visual>
         <origin xyz="0 0 0" rpy="0 0 0"/>
         <geometry>
-          <mesh filename="package://barista_description/meshes/barista/bowtie_fixed_colour.dae"/>
+          <xacro:if value="${robot_name_prop == 'barista_1'}">
+            <mesh filename="package://barista_description/meshes/barista/BOTTOM_colour_1.dae"/>
+          </xacro:if>
+          <xacro:if value="${robot_name_prop == 'barista_2'}">
+            <mesh filename="package://barista_description/meshes/barista/BOTTOM_colour_2.dae"/>
+          </xacro:if>
+          <xacro:if value="${robot_name_prop != 'barista_1' and robot_name_prop != 'barista_2'}">
+            <mesh filename="package://barista_description/meshes/barista/BOTTOM_colour.dae"/>
+          </xacro:if>
         </geometry>
       </visual>
       <collision>
-        <origin xyz="-0.0294981 0.0 0.0" rpy="0 0 0"/>
+        <origin xyz="0 0 -0.07" rpy="0 0 0"/>
         <geometry>
-          <box size="0.115703 0.024221 0.0589962"/>
+          <cylinder length="0.14" radius="0.1760015"/>
         </geometry>
       </collision>
       <inertial>
-        <mass value="0.01" />
+        <mass value="0.1" />
         <origin xyz="0 0 0" />
-        <inertia ixx="3.38934037953e-06" ixy="0.0" ixz="0.0"
-                 iyy="1.40564465195e-05" iyz="0.0"
-                 izz="1.16448675417e-05" />
+        <inertia ixx="0.00093774653339" ixy="0.0" ixz="0.0"
+                 iyy="0.00093774653339" iyz="0.0"
+                 izz="0.00154882640011" />
       </inertial>
     </link>
-    <joint name="barista_bowtie_joint" type="fixed">
-      <origin xyz="0.195852 0.0 0.01874" rpy="0 0 1.57"/>
-      <parent link="barista_top_link"/>
-      <child link="barista_bowtie_link"/>
+    <joint name="barista_bottom_joint" type="fixed">
+      <origin xyz="0.01 0.0 0.0" rpy="0 0 0"/>
+      <parent link="${bottom_parent}"/>
+      <child link="barista_bottom_link"/>
+    </joint>
+  </xacro:macro>
+  <!-- Mule Related -->
+  <xacro:macro name="barista_mod_mule" params="bottom_parent top_parent">
+    <link name="barista_top_link">
+      <visual>
+        <origin xyz="0 0 0" rpy="0 0 0"/>
+        <geometry>
+          <mesh filename="package://barista_description/meshes/barista/TOP_mule.dae"/>
+        </geometry>
+      </visual>
+      <collision>
+        <origin xyz="0 0 0" rpy="0 0 0"/>
+        <geometry>
+          <mesh filename="package://barista_description/meshes/barista/TOP_mule_col.stl"/>
+        </geometry>
+      </collision>
+      <inertial>
+        <mass value="0.1" />
+        <origin xyz="0 0 0" />
+        <inertia ixx="0.00083462153339" ixy="0.0" ixz="0.0"
+                 iyy="0.00083462153339" iyz="0.0"
+                 izz="0.00154882640011" />
+      </inertial>
+    </link>
+    <joint name="barista_top_joint" type="fixed">
+      <origin xyz="0.01 0.0 0.09" rpy="0 0 0"/>
+      <parent link="${top_parent}"/>
+      <child link="barista_top_link"/>
     </joint>
     <link name="barista_bottom_link">
@@ -62,5 +107,5 @@
         <origin xyz="0 0 0" rpy="0 0 0"/>
         <geometry>
-          <mesh filename="package://barista_description/meshes/barista/BOTTOM_colour.dae"/>
+          <mesh filename="package://barista_description/meshes/barista/BOTTOM_mule.dae"/>
         </geometry>
       </visual>

Commit message: Added corrected centers adn scales of meshes for gzweb to work

File: barista_description/robot/barista_hexagons.xacro (robot description, xacro)
@@ -19,5 +19,5 @@
         <origin xyz="0 0 0" rpy="0 0 0"/>
         <geometry>
-          <mesh filename="package://barista_description/meshes/turtlebot/stacks/hexagons/pole_bottom.dae"/>
+          <mesh filename="package://barista_description/meshes/turtlebot/stacks/hexagons/pole_bottom_v2.dae"/>
         </geometry>
       </visual>
@@ -47,5 +47,5 @@
         <origin xyz="0 0 0" rpy="0 ${M_PI} 0"/>
         <geometry>
-          <mesh filename="package://barista_description/meshes/turtlebot/stacks/hexagons/pole_middle.dae"/>
+          <mesh filename="package://barista_description/meshes/turtlebot/stacks/hexagons/pole_middle_v2.dae"/>
         </geometry>
       </visual>
@@ -75,5 +75,5 @@
         <origin xyz=" 0 0 0" rpy="0 0 0"/>
         <geometry>
-          <mesh filename="package://barista_description/meshes/turtlebot/stacks/hexagons/pole_top.dae"/>
+          <mesh filename="package://barista_description/meshes/turtlebot/stacks/hexagons/pole_top_v2.dae"/>
         </geometry>
       </visual>
@@ -178,5 +178,5 @@
         <origin xyz="0 0 0" rpy="0 0 0"/>
         <geometry>
-          <mesh filename="package://barista_description/meshes/turtlebot/stacks/hexagons/plate_bottom.dae"/>
+          <mesh filename="package://barista_description/meshes/turtlebot/stacks/hexagons/plate_bottom_v2.dae"/>
         </geometry>
       </visual>
@@ -208,5 +208,5 @@
         <origin xyz="0 0 0" rpy="0 0 0"/>
         <geometry>
-          <mesh filename="package://barista_description/meshes/turtlebot/stacks/hexagons/plate_middle.dae"/>
+          <mesh filename="package://barista_description/meshes/turtlebot/stacks/hexagons/plate_middle_v2.dae"/>
         </geometry>
       </visual>
