Commit message: Added corrections to make barista with three robots dont fail as often and optimization for speed

File: barista_description/robot/barista_hokuyo.xacro (robot description, xacro)
@@ -35,5 +35,5 @@
   		<sensor name="lidar" type="ray">
 			<always_on>true</always_on>
-			<visualize>false</visualize>
+			<visualize>true</visualize>
 			<update_rate>20</update_rate>
 			<ray>
@@ -67,28 +67,4 @@
 		</sensor>
   	</gazebo>
-	<gazebo>
-		<plugin name='diff_drive' filename='libgazebo_ros_diff_drive.so'>
-			<ros>
-				<namespace>/</namespace>
-				<argument>cmd_vel:=${robot_name}/cmd_vel</argument>
-				<argument>odom:=${robot_name}/odom</argument>
-			</ros>
-			<!-- wheels -->
-			<left_joint>${robot_name}/joint_tire_left</left_joint>
-			<right_joint>${robot_name}/joint_tire_right</right_joint>
-			<!-- kinematics -->
-			<wheel_separation>0.4</wheel_separation>
-			<wheel_diameter>0.1</wheel_diameter>
-			<!-- limits -->
-			<max_wheel_torque>20</max_wheel_torque>
-			<max_wheel_acceleration>1.0</max_wheel_acceleration>
-			<!-- output -->
-			<publish_odom>true</publish_odom>
-			<publish_odom_tf>true</publish_odom_tf>
-			<publish_wheel_tf>false</publish_wheel_tf>
-			<odometry_frame>${robot_name}/odom</odometry_frame>
-			<robot_base_frame>${robot_name}/base_footprint</robot_base_frame>
-		</plugin>
-	</gazebo>
   </xacro:macro>
 </robot>

File: barista_description/robot/barista_kobuki_gazebo.xacro (robot description, xacro)
@@ -137,4 +137,28 @@
       </sensor>
 	  </gazebo>
+	<gazebo>
+		<plugin name='diff_drive' filename='libgazebo_ros_diff_drive.so'>
+			<ros>
+				<namespace>/</namespace>
+				<argument>cmd_vel:=${robot_name}/cmd_vel</argument>
+				<argument>odom:=${robot_name}/odom</argument>
+			</ros>
+			<!-- wheels -->
+			<left_joint>${robot_name}/joint_tire_left</left_joint>
+			<right_joint>${robot_name}/joint_tire_right</right_joint>
+			<!-- kinematics -->
+			<wheel_separation>0.4</wheel_separation>
+			<wheel_diameter>0.1</wheel_diameter>
+			<!-- limits -->
+			<max_wheel_torque>20</max_wheel_torque>
+			<max_wheel_acceleration>1.0</max_wheel_acceleration>
+			<!-- output -->
+			<publish_odom>true</publish_odom>
+			<publish_odom_tf>true</publish_odom_tf>
+			<publish_wheel_tf>false</publish_wheel_tf>
+			<odometry_frame>${robot_name}/odom</odometry_frame>
+			<robot_base_frame>${robot_name}/base_footprint</robot_base_frame>
+		</plugin>
+	</gazebo>
   </xacro:macro>
 </robot>

File: barista_description/robot/barista_mod copy.xacro (robot description, xacro)
@@ -24,5 +24,6 @@
         <origin xyz="0 0 0" rpy="0 0 0"/>
         <geometry>
-          <mesh filename="package://barista_description/meshes/barista/TOP_collision_lip_sd.stl"/>
+          <mesh filename="package://barista_description/meshes/barista/TOP_collision_lip.stl"/>
+          <!-- <cylinder length="0.085" radius="0.1760015"/> -->
         </geometry>
       </collision>
@@ -55,4 +56,10 @@
         </geometry>
       </visual>
+      <collision>
+        <origin xyz="0 0 -0.07" rpy="0 0 0"/>
+        <geometry>
+          <cylinder length="0.14" radius="0.1760015"/>
+        </geometry>
+      </collision>
       <inertial>
         <mass value="0.1" />
@@ -64,5 +71,5 @@
     </link>
     <joint name="barista_bottom_joint" type="fixed">
-      <origin xyz="0.001 0.0 0.12" rpy="0 0 0"/>
+      <origin xyz="-0.00364 0.0 0.1874" rpy="0 0 0"/>
       <parent link="${bottom_parent}"/>
       <child link="barista_bottom_link"/>
@@ -81,5 +88,5 @@
         <origin xyz="0 0 0" rpy="0 0 0"/>
         <geometry>
-          <mesh filename="package://barista_description/meshes/barista/TOP_mule_col_sd.stl"/>
+          <mesh filename="package://barista_description/meshes/barista/TOP_mule_col.stl"/>
         </geometry>
       </collision>
@@ -93,5 +100,5 @@
     </link>
     <joint name="barista_top_joint" type="fixed">
-      <origin xyz="0.00364 0.0 0.24583" rpy="0 0 0"/>
+      <origin xyz="0.00364 0.0 0.3966" rpy="0 0 0"/>
       <parent link="${top_parent}"/>
       <child link="barista_top_link"/>
@@ -104,4 +111,10 @@
         </geometry>
       </visual>
+      <collision>
+        <origin xyz="0 0 -0.07" rpy="0 0 0"/>
+        <geometry>
+          <cylinder length="0.14" radius="0.1760015"/>
+        </geometry>
+      </collision>
       <inertial>
         <mass value="0.1" />
@@ -113,5 +126,5 @@
     </link>
     <joint name="barista_bottom_joint" type="fixed">
-      <origin xyz="0.001 0.0 0.12" rpy="0 0 0"/>
+      <origin xyz="-0.00364 0.0 0.1874" rpy="0 0 0"/>
       <parent link="${bottom_parent}"/>
       <child link="barista_bottom_link"/>

File: barista_description/robot/mule_barista copy.xacro (robot description, xacro)
@@ -7,13 +7,17 @@
   <!-- Bases -->
   <xacro:include filename="$(find barista_description)/robot/barista_kobuki.xacro" />
+  <!-- Stacks -->
+  <xacro:include filename="$(find barista_description)/robot/barista_hexagons.xacro"/>
   <xacro:include filename="$(find barista_description)/robot/barista_mod.xacro" />
   <xacro:include filename="$(find barista_description)/robot/barista_hokuyo.xacro" />
   <xacro:barista_kobuki robot_name="$(arg robot_name)"/>
   <xacro:if value="${'barista' in robot_name_prop}">
-    <xacro:barista_mod  bottom_parent="base_link" top_parent="base_link"/>
+    <xacro:stack_hexagons parent="base_link"/>
+    <xacro:barista_mod  bottom_parent="plate_middle_link" top_parent="plate_top_link"/>
   </xacro:if>
   <xacro:if value="${'mule' in robot_name_prop}">
-    <xacro:barista_mod_mule  bottom_parent="base_link" top_parent="base_link"/>
+    <xacro:stack_hexagons_mule parent="base_link"/>
+    <xacro:barista_mod_mule  bottom_parent="plate_middle_link" top_parent="plate_middle_link"/>
   </xacro:if>
-  <xacro:barista_hokuyo  parent="base_link" x_hok="0.103007" y_hok="0.0" z_hok="0.17" robot_name="$(arg robot_name)"/>
+  <xacro:barista_hokuyo  parent="plate_middle_link" x_hok="0.116647" y_hok="0.0" z_hok="0.045" robot_name="$(arg robot_name)"/>
 </robot>

Commit message: Added simpler meshes, no laser vis and barstools without nav

File: barista_description/robot/barista_hokuyo.xacro (robot description, xacro)
@@ -35,5 +35,5 @@
   		<sensor name="lidar" type="ray">
 			<always_on>true</always_on>
-			<visualize>true</visualize>
+			<visualize>false</visualize>
 			<update_rate>20</update_rate>
 			<ray>

File: barista_description/robot/barista_kobuki.xacro (robot description, xacro)
@@ -37,9 +37,9 @@
     <joint name="${robot_name}/joint_tire_left" type="continuous">
     <parent link="base_link"/>
-    <child link="wheel_left_link"/>
+    <child link="${robot_name}/wheel_left_link"/>
     <origin rpy="-1.5707963267948966 0 0" xyz="0.00 0.115 0.0250"/>
     <axis xyz="0 0 1"/>
   </joint>
-  <link name="wheel_left_link">
+  <link name="${robot_name}/wheel_left_link">
     <visual>
       <geometry>
@@ -62,9 +62,9 @@
   <joint name="${robot_name}/joint_tire_right" type="continuous">
     <parent link="base_link"/>
-    <child link="wheel_right_link"/>
+    <child link="${robot_name}/wheel_right_link"/>
     <origin rpy="-1.5707963267948966 0 0" xyz="0.00 -0.115 0.0250"/>
     <axis xyz="0 0 1"/>
   </joint>
-  <link name="wheel_right_link">
+  <link name="${robot_name}/wheel_right_link">
     <visual>
       <geometry>

File: barista_description/robot/barista_kobuki_gazebo.xacro (robot description, xacro)
@@ -51,5 +51,5 @@
 	      <always_on>true</always_on>
 	      <update_rate>50</update_rate>
-	      <visualize>false</visualize>
+	      <visualize>true</visualize>
 	      <ray>
 	        <scan>
@@ -73,5 +73,5 @@
 	      <always_on>true</always_on>
 	      <update_rate>50</update_rate>
-	      <visualize>false</visualize>
+	      <visualize>true</visualize>
 	      <ray>
 	        <scan>
@@ -95,5 +95,5 @@
 	      <always_on>true</always_on>
 	      <update_rate>50</update_rate>
-	      <visualize>false</visualize>
+	      <visualize>true</visualize>
 	      <ray>
 	        <scan>

Commit message: first commit

File: barista_description/robot/barista_hokuyo.xacro (robot description, xacro)
@@ -40,5 +40,5 @@
 				<scan>
 					<horizontal>
-					<samples>128</samples>
+					<samples>720</samples>
 					<resolution>1.000000</resolution>
 					<min_angle>0.000000</min_angle>
@@ -48,5 +48,5 @@
 				<range>
 					<min>0.120000</min>
-					<max>3.5</max>
+					<max>6.0</max>
 					<resolution>0.015000</resolution>
 				</range>

File: barista_description/robot/barista_kobuki.xacro (robot description, xacro)
@@ -35,11 +35,11 @@
       </inertial>
     </link>
-    <joint name="${robot_name}/joint_tire_left" type="continuous">
+    <joint name="joint_tire_left" type="continuous">
     <parent link="base_link"/>
-    <child link="${robot_name}/wheel_left_link"/>
+    <child link="wheel_left_link"/>
     <origin rpy="-1.5707963267948966 0 0" xyz="0.00 0.115 0.0250"/>
     <axis xyz="0 0 1"/>
   </joint>
-  <link name="${robot_name}/wheel_left_link">
+  <link name="wheel_left_link">
     <visual>
       <geometry>
@@ -60,11 +60,11 @@
     </inertial>
   </link>
-  <joint name="${robot_name}/joint_tire_right" type="continuous">
+  <joint name="joint_tire_right" type="continuous">
     <parent link="base_link"/>
-    <child link="${robot_name}/wheel_right_link"/>
+    <child link="wheel_right_link"/>
     <origin rpy="-1.5707963267948966 0 0" xyz="0.00 -0.115 0.0250"/>
     <axis xyz="0 0 1"/>
   </joint>
-  <link name="${robot_name}/wheel_right_link">
+  <link name="wheel_right_link">
     <visual>
       <geometry>

File: barista_description/robot/barista_kobuki_gazebo.xacro (robot description, xacro)
@@ -145,6 +145,6 @@
 			</ros>
 			<!-- wheels -->
-			<left_joint>${robot_name}/joint_tire_left</left_joint>
-			<right_joint>${robot_name}/joint_tire_right</right_joint>
+			<left_joint>joint_tire_left</left_joint>
+			<right_joint>joint_tire_right</right_joint>
 			<!-- kinematics -->
 			<wheel_separation>0.4</wheel_separation>
